File: schematics/PlytkaProcesor.brd (EAGLE design)
At the start: 70 x 70 mm, 56 parts, among them IC1 FM24CL64B-GTR, IC2 SCD40-D-R1, IC3 NRF52840-QIAA-R, J1 F34G-1A7Q1-E8C24, Q1 PMOSFET, Q3 PMOSFET, Q5 PMOSFET, Q6 NMOSFET, Q7 NMOSFET

Commit message: Project Final
Parts:
- removed D1: LED_RED, LED:LEDC1608X35N_FLAT-R
- removed R7: 220, Resistor:RESC1005X40
- added C8: 0.1uF, Capacitor:CAPC1608X85
- added U$1: N0M59S10IC, N0M59S10IC:N0M59S10IC
Connections:
- removed net N$1: D1.A, R7.2
- net 3V3: now also C8.1, U$1.VDD
- net D2: now also U$1.DIN; no longer R7.1
- net GND: now also C8.2, U$1.VSS; no longer D1.C
Routing:
- net 3V3: track 184.7 -> 202.3 mm
- net N$1: track 9.78 -> 0.00 mm
- net D2: track 31.3 -> 35.3 mm
Changed lines of the file:
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@@
 <plain>
 <circle x="0.5" y="-0.5045" radius="35" width="0.1524" layer="20"/>
+<polygon width="0.1524" layer="1" pour="cutout">
+<vertex x="-34.9758" y="17.3482"/>
+<vertex x="-23.9075625" y="17.3482"/>
+<vertex x="-23.2841625" y="17.9716"/>
+<vertex x="-23.25615625" y="17.9832"/>
+<vertex x="-22.2565625" y="17.9832"/>
+<vertex x="-19.5072" y="20.7325625"/>
+<vertex x="-19.5072" y="22.4474375"/>
+<vertex x="-24.4155625" y="27.3558"/>
+<vertex x="-34.8934375" y="27.3558"/>
+<vertex x="-34.9758" y="27.2734375"/>
+</polygon>
+<polygon width="0.1524" layer="16" pour="cutout">
+<vertex x="-34.9758" y="17.3482"/>
+<vertex x="-23.9075625" y="17.3482"/>
+<vertex x="-23.2841625" y="17.9716"/>
+<vertex x="-23.25615625" y="17.9832"/>
+<vertex x="-22.2565625" y="17.9832"/>
+<vertex x="-19.5072" y="20.7325625"/>
+<vertex x="-19.5072" y="22.4474375"/>
+<vertex x="-24.4155625" y="27.3558"/>
+<vertex x="-34.8934375" y="27.3558"/>
+<vertex x="-34.9758" y="27.2734375"/>
+</polygon>
 </plain>
 <attributes>
@@
 <attribute name="VALUE" x="0.374" y="-25.171" size="1.27" layer="27" align="center"/>
 </element>
-<element name="D1" library="LED" package="LEDC1608X35N_FLAT-R" package3d_urn="urn:adsk.eagle:package:24294797/1" value="LED_RED" x="0.237" y="-31.575" smashed="yes">
-<attribute name="CATEGORY" value="LED" x="0.237" y="-31.575" size="1.778" layer="27" display="off"/>
-<attribute name="COLOR" value="RED" x="0.237" y="-31.575" size="1.778" layer="27" display="off"/>
-<attribute name="DESCRIPTION" value="CHIP LED FLAT" x="0.237" y="-31.575" size="1.778" layer="27" display="off"/>
-<attribute name="MANUFACTURER" value="" x="0.237" y="-31.575" size="1.778" layer="27" display="off"/>
-<attribute name="MPN" value="" x="0.237" y="-31.575" size="1.778" layer="27" display="off"/>
-<attribute name="NAME" x="0.11" y="-30.1701" size="1.27" layer="25" align="bottom-center"/>
-<attribute name="OPERATING_TEMP" value="" x="0.237" y="-31.575" size="1.778" layer="27" display="off"/>
-<attribute name="PART_STATUS" value="" x="0.237" y="-31.575" size="1.778" layer="27" display="off"/>
-<attribute name="ROHS_COMPLIANT" value="" x="0.237" y="-31.575" size="1.778" layer="27" display="off"/>
-<attribute name="SERIES" value="" x="0.237" y="-31.575" size="1.778" layer="27" display="off"/>
-<attribute name="SUB-CATEGORY" value="CHIP" x="0.237" y="-31.575" size="1.778" layer="27" display="off"/>
-<attribute name="THERMALLOSS" value="" x="0.237" y="-31.575" size="1.778" layer="27" display="off"/>
-<attribute name="TYPE" value="FLAT_TOP" x="0.237" y="-31.575" size="1.778" layer="27" display="off"/>
-<attribute name="VALUE" x="0.11" y="-32.9799" size="1.27" layer="27" align="top-center"/>
-</element>
 <element name="H3" library="holes" library_urn="urn:adsk.eagle:library:237" package="2,8" package3d_urn="urn:adsk.eagle:package:14271/1" value="MOUNT-HOLE2.8" x="-19.568" y="-13.292" smashed="yes">
 <attribute name="POPULARITY" value="15" x="-19.568" y="-13.292" size="1.778" layer="27" display="off"/>
@@
 <attribute name="VALUE" x="-17.234" y="0.286" size="1.27" layer="27" rot="R270" align="center"/>
 </element>
-<element name="R7" library="Resistor" package="RESC1005X40" package3d_urn="urn:adsk.eagle:package:16378568/2" value="220" x="10.16" y="-29.591" smashed="yes" rot="R270">
-<attribute name="CATEGORY" value="Resistor" x="10.16" y="-31.623" size="1.778" layer="27" rot="R270" display="off"/>
-<attribute name="MANUFACTURER" value="" x="10.16" y="-31.623" size="1.778" layer="27" rot="R270" display="off"/>
-<attribute name="MPN" value="" x="10.16" y="-31.623" size="1.778" layer="27" rot="R270" display="off"/>
-<attribute name="NAME" x="11.431" y="-29.591" size="1.27" layer="25" rot="R270" align="bottom-center"/>
-<attribute name="OPERATING_TEMP" value="" x="10.16" y="-31.623" size="1.778" layer="27" rot="R270" display="off"/>
-<attribute name="PART_STATUS" value="" x="10.16" y="-31.623" size="1.778" layer="27" rot="R270" display="off"/>
-<attribute name="RATING" value="" x="10.16" y="-31.623" size="1.778" layer="27" rot="R270" display="off"/>
-<attribute name="ROHS_COMPLIANT" value="" x="10.16" y="-31.623" size="1.778" layer="27" rot="R270" display="off"/>
-<attribute name="SERIES" value="" x="10.16" y="-31.623" size="1.778" layer="27" rot="R270" display="off"/>
-<attribute name="SUB-CATEGORY" value="Fixed" x="10.16" y="-31.623" size="1.778" layer="27" rot="R270" display="off"/>
-<attribute name="THERMALLOSS" value="" x="10.16" y="-31.623" size="1.778" layer="27" rot="R270" display="off"/>
-<attribute name="TOLERANCE" value="" x="10.16" y="-31.623" size="1.778" layer="27" rot="R270" display="off"/>
-<attribute name="TYPE" value="" x="10.16" y="-31.623" size="1.778" layer="27" rot="R270" display="off"/>
-<attribute name="VALUE" x="8.889" y="-29.591" size="1.27" layer="27" rot="R270" align="top-center"/>
+<element name="U$1" library="N0M59S10IC" library_urn="urn:adsk.wipprod:fs.file:vf.S77eDUjJS8qFZARyPbMuKQ" package="N0M59S10IC" value="N0M59S10IC" x="-0.381" y="-32.639" smashed="yes"/>
+<element name="C8" library="Capacitor" package="CAPC1608X85" package3d_urn="urn:adsk.eagle:package:16290898/2" value="0.1uF" x="12.319" y="-27.813" smashed="yes" rot="R270">
+<attribute name="CATEGORY" value="Capacitor" x="12.319" y="-29.21" size="1.778" layer="27" rot="R270" display="off"/>
+<attribute name="MANUFACTURER" value="" x="12.319" y="-29.21" size="1.778" layer="27" rot="R270" display="off"/>
+<attribute name="MPN" value="" x="12.319" y="-29.21" size="1.778" layer="27" rot="R270" display="off"/>
+<attribute name="NAME" x="13.7531" y="-27.813" size="1.27" layer="25" rot="R270" align="bottom-center"/>
+<attribute name="OPERATING_TEMP" value="" x="12.319" y="-29.21" size="1.778" layer="27" rot="R270" display="off"/>
+<attribute name="PART_STATUS" value="" x="12.319" y="-29.21" size="1.778" layer="27" rot="R270" display="off"/>
+<attribute name="ROHS_COMPLIANT" value="" x="12.319" y="-29.21" size="1.778" layer="27" rot="R270" display="off"/>
+<attribute name="SERIES" value="" x="12.319" y="-29.21" size="1.778" layer="27" rot="R270" display="off"/>
+<attribute name="SUB-CATEGORY" value="" x="12.319" y="-29.21" size="1.778" layer="27" rot="R270" display="off"/>
+<attribute name="THERMALLOSS" value="" x="12.319" y="-29.21" size="1.778" layer="27" rot="R270" display="off"/>
+<attribute name="TYPE" value="" x="12.319" y="-29.21" size="1.778" layer="27" rot="R270" display="off"/>
+<attribute name="VALUE" x="10.8849" y="-27.813" size="1.27" layer="27" rot="R270" align="top-center"/>
+<attribute name="VOLTAGE_RATING" value="" x="12.319" y="-29.21" size="1.778" layer="27" rot="R270" display="off"/>
 </element>
 </elements>
@@
 <contactref element="JP3" pad="5"/>
 <contactref element="S1" pad="1"/>
-<contactref element="D1" pad="C"/>
 <contactref element="J1" pad="8"/>
 <contactref element="J1" pad="17"/>
@@
 <wire x1="4.16696875" y1="29.8704" x2="4.39556875" y2="30.099" width="0.6096" layer="1"/>
 <wire x1="4.39556875" y1="30.099" x2="4.699" y2="30.099" width="0.6096" layer="1"/>
+<contactref element="U$1" pad="VSS"/>
+<contactref element="C8" pad="2"/>
 </signal>
 <signal name="N$5">
@@
 <wire x1="15.97536875" y1="23.458" x2="9.3240625" y2="23.458" width="1.016" layer="16"/>
 <wire x1="9.3240625" y1="23.458" x2="2.3114" y2="30.4706625" width="1.016" layer="16"/>
+<contactref element="U$1" pad="VDD"/>
+<contactref element="C8" pad="1"/>
+<wire x1="10.414" y1="-23.8765" x2="11.0495" y2="-23.8765" width="0.4064" layer="1"/>
+<wire x1="11.0495" y1="-23.8765" x2="12.319" y2="-25.146" width="0.4064" layer="1"/>
+<wire x1="12.319" y1="-25.146" x2="12.319" y2="-27.0384" width="0.4064" layer="1"/>
+<wire x1="0.769" y1="-31.239" x2="8.1184" y2="-31.239" width="0.4064" layer="1"/>
+<wire x1="8.1184" y1="-31.239" x2="12.319" y2="-27.0384" width="0.4064" layer="1"/>
 </signal>
 <signal name="N$4">
@@
 <wire x1="0.6071" y1="-14.7283" x2="0.4287" y2="-14.9067" width="0.3048" layer="1"/>
 <via x="0.4287" y="-14.9067" extent="1-16" drill="0.35"/>
-<contactref element="R7" pad="1"/>
-<via x="9.906" y="-28.194" extent="1-16" drill="0.35"/>
-<wire x1="9.906" y1="-28.194" x2="10.16" y2="-28.448" width="0.3048" layer="1"/>
-<wire x1="10.16" y1="-28.448" x2="10.16" y2="-29.0835" width="0.3048" layer="1"/>
 <wire x1="0.4287" y1="-14.9067" x2="4.38085" y2="-18.85885" width="0.3048" layer="16"/>
-<wire x1="4.38085" y1="-18.85885" x2="4.38085" y2="-22.66885" width="0.3048" layer="16"/>
-<wire x1="4.38085" y1="-22.66885" x2="9.906" y2="-28.194" width="0.3048" layer="16"/>
+<contactref element="U$1" pad="DIN"/>
+<wire x1="4.38085" y1="-18.85885" x2="4.38085" y2="-31.56015" width="0.3048" layer="16"/>
+<wire x1="4.38085" y1="-31.56015" x2="3.556" y2="-32.385" width="0.3048" layer="16"/>
+<via x="3.556" y="-32.385" extent="1-16" drill="0.35"/>
+<wire x1="3.556" y1="-32.385" x2="3.502" y2="-32.439" width="0.3048" layer="1"/>
+<wire x1="3.502" y1="-32.439" x2="0.769" y2="-32.439" width="0.3048" layer="1"/>
 </signal>
 <signal name="VPP">
 <contactref element="J1" pad="6"/>
 </signal>
-<signal name="N$1">
-<contactref element="D1" pad="A"/>
-<contactref element="R7" pad="2"/>
-<wire x1="10.16" y1="-30.0985" x2="8.6835" y2="-31.575" width="0.3048" layer="1"/>
-<wire x1="8.6835" y1="-31.575" x2="0.987" y2="-31.575" width="0.3048" layer="1"/>
-</signal>
 </signals>
