File: schematics/SchematProcesor.sch (EAGLE design)
At the start: 56 parts, among them IC1 FM24CL64B-GTR, IC2 SCD40-D-R1, IC3 NRF52840-QIAA-R, J1 F34G-1A7Q1-E8C24, Q1 PMOSFET, Q3 PMOSFET, Q5 PMOSFET, Q6 NMOSFET, Q7 NMOSFET

Commit message: Project Final
Parts:
- removed D1: LED_RED, LED:CHIP-FLAT-R_0603-0.35MM
- removed R7: 220, Resistor:R_CHIP-0402(1005-METRIC)
- added C8: 0.1uF, Capacitor:C_CHIP-0603(1608-METRIC)
- added U$1: N0M59S10IC, N0M59S10IC:N0M59S10IC
Connections:
- removed net N$1: D1.A, R7.2
- net 3V3: now also C8.1, U$1.VDD
- net D2: now also U$1.DIN; no longer R7.1
- net GND: now also C8.2, U$1.VSS; no longer D1.C
Changed lines of the file:
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@@
 <part name="JP3" library="Connector" deviceset="PINHD-1X5" device="" package3d_urn="urn:adsk.eagle:package:22469/2"/>
 <part name="S1" library="SamacSys_Parts" deviceset="MX1A-C1NN" device=""/>
-<part name="D1" library="LED" deviceset="CHIP-FLAT-R" device="_0603-0.35MM" package3d_urn="urn:adsk.eagle:package:24294797/1" value="LED_RED"/>
 <part name="H3" library="holes" library_urn="urn:adsk.eagle:library:237" deviceset="MOUNT-HOLE" device="2.8" package3d_urn="urn:adsk.eagle:package:14271/1"/>
 <part name="H4" library="holes" library_urn="urn:adsk.eagle:library:237" deviceset="MOUNT-HOLE" device="2.8" package3d_urn="urn:adsk.eagle:package:14271/1"/>
 <part name="J1" library="Biblioteka" library_urn="urn:adsk.wipprod:fs.file:vf.O-cfOsubQTu2HNn45N_EGQ" deviceset="F34G-1A7Q1-E8C24" device=""/>
-<part name="R7" library="Resistor" deviceset="R" device="CHIP-0402(1005-METRIC)" package3d_urn="urn:adsk.eagle:package:16378568/2" technology="_" value="220"/>
+<part name="U$1" library="N0M59S10IC" library_urn="urn:adsk.wipprod:fs.file:vf.S77eDUjJS8qFZARyPbMuKQ" deviceset="N0M59S10IC" device=""/>
+<part name="C8" library="Capacitor" deviceset="C" device="CHIP-0603(1608-METRIC)" package3d_urn="urn:adsk.eagle:package:16290898/2" technology="_" value="0.1uF"/>
+<part name="SUPPLY25" library="Power_Symbols" deviceset="GND-EARTH" device="" value="GND"/>
 </parts>
 <sheets>
@@
 <attribute name="VALUE" x="219.71" y="157.48" size="1.778" layer="96" align="center-left"/>
 </instance>
-<instance part="D1" gate="G$1" x="218.44" y="142.24" smashed="yes" rot="R270">
-<attribute name="NAME" x="220.98" y="137.922" size="1.778" layer="95" align="top-right"/>
-<attribute name="VALUE" x="220.98" y="140.462" size="1.778" layer="96" align="top-right"/>
-</instance>
 <instance part="H3" gate="G$1" x="228.6" y="76.2" smashed="yes">
 <attribute name="NAME" x="230.632" y="76.7842" size="1.778" layer="95"/>
@@
 <attribute name="VALUE" x="230.632" y="66.1162" size="1.778" layer="96"/>
 </instance>
-<instance part="R7" gate="G$1" x="228.6" y="142.24" smashed="yes" rot="R180">
-<attribute name="NAME" x="228.6" y="139.7" size="1.778" layer="95" rot="R180" align="center"/>
-<attribute name="VALUE" x="228.6" y="144.78" size="1.778" layer="96" rot="R180" align="center"/>
+<instance part="U$1" gate="G$1" x="223.52" y="137.16" smashed="yes"/>
+<instance part="C8" gate="G$1" x="246.38" y="134.62" smashed="yes">
+<attribute name="NAME" x="248.92" y="134.62" size="1.778" layer="95"/>
+<attribute name="VALUE" x="248.92" y="132.08" size="1.778" layer="96"/>
+</instance>
+<instance part="SUPPLY25" gate="G$1" x="246.38" y="124.46" smashed="yes">
+<attribute name="VALUE" x="246.38" y="121.285" size="1.778" layer="96" align="center"/>
 </instance>
 </instances>
@@
 <junction x="231.14" y="124.46"/>
 <label x="226.06" y="124.46" size="1.778" layer="95"/>
+</segment>
+<segment>
+<pinref part="U$1" gate="G$1" pin="VDD"/>
+<wire x1="243.84" y1="139.7" x2="246.38" y2="139.7" width="0.1524" layer="91"/>
+<label x="248.92" y="139.7" size="1.778" layer="95"/>
+<wire x1="246.38" y1="139.7" x2="248.92" y2="139.7" width="0.1524" layer="91"/>
+<junction x="246.38" y="139.7"/>
+<wire x1="246.38" y1="139.7" x2="246.38" y2="137.16" width="0.1524" layer="91"/>
+<pinref part="C8" gate="G$1" pin="1"/>
 </segment>
 </net>
@@
 </segment>
 <segment>
-<wire x1="210.82" y1="152.4" x2="210.82" y2="142.24" width="0.1524" layer="91"/>
+<wire x1="210.82" y1="152.4" x2="210.82" y2="144.78" width="0.1524" layer="91"/>
 <pinref part="SUPPLY5" gate="G$1" pin="GND"/>
 <pinref part="S1" gate="G$1" pin="1"/>
-<wire x1="210.82" y1="142.24" x2="210.82" y2="137.16" width="0.1524" layer="91"/>
+<wire x1="210.82" y1="144.78" x2="210.82" y2="137.16" width="0.1524" layer="91"/>
 <wire x1="218.44" y1="152.4" x2="210.82" y2="152.4" width="0.1524" layer="91"/>
-<pinref part="D1" gate="G$1" pin="C"/>
-<wire x1="213.36" y1="142.24" x2="210.82" y2="142.24" width="0.1524" layer="91"/>
-<junction x="210.82" y="142.24"/>
+<pinref part="U$1" gate="G$1" pin="VSS"/>
+<wire x1="218.44" y1="144.78" x2="210.82" y2="144.78" width="0.1524" layer="91"/>
+<junction x="210.82" y="144.78"/>
+</segment>
+<segment>
+<pinref part="C8" gate="G$1" pin="2"/>
+<wire x1="246.38" y1="129.54" x2="246.38" y2="127" width="0.1524" layer="91"/>
+<pinref part="SUPPLY25" gate="G$1" pin="GND"/>
 </segment>
 </net>
@@
 </segment>
 <segment>
-<pinref part="R7" gate="G$1" pin="1"/>
-<wire x1="233.68" y1="142.24" x2="238.76" y2="142.24" width="0.1524" layer="91"/>
-<label x="238.76" y="142.24" size="1.778" layer="95"/>
-</segment>
-</net>
-<net name="N$1" class="0">
-<segment>
-<pinref part="D1" gate="G$1" pin="A"/>
-<wire x1="220.98" y1="142.24" x2="223.52" y2="142.24" width="0.1524" layer="91"/>
-<pinref part="R7" gate="G$1" pin="2"/>
-</segment>
-</net>
+<pinref part="U$1" gate="G$1" pin="DIN"/>
+<wire x1="243.84" y1="144.78" x2="248.92" y2="144.78" width="0.1524" layer="91"/>
+<label x="248.92" y="144.78" size="1.778" layer="95"/>
+</segment>
+</net>
